Commit message: add world launch file

File: robot_description/urdf/my_robot.xacro (robot description, xacro)
@@ -4,5 +4,5 @@
     <xacro:include filename="$(find robot_description)/my_robot_lidar.xacro" />
     <joint name="lidar_joint" type="fixed">
-        <origin xyz="${base_radius-lidar_radius} 0 ${base_length+wheel_radius/3}" rpy="0 0 0" />
+        <origin xyz="${-base_radius+lidar_radius} 0 ${base_length+wheel_radius/3}" rpy="0 0 ${PI}" />
         <parent link="base_link" />
         <child link="lidar_link" />

File: robot_description/urdf/sensors/my_robot_lidar.xacro (robot description, xacro)
@@ -32,5 +32,5 @@
             <sensor type="ray" name="head_hokuyo_sensor">
                 <visualize>true</visualize>
-                <update_rate>10</update_rate>
+                <update_rate>2</update_rate>
                 <ray>
                     <scan>
@@ -56,5 +56,5 @@
                     <ros>
                         <namespace>/</namespace>
-                        <argument>--ros-args --remap out:=scan</argument>
+                        <argument>~/out:=/scan</argument>
                     </ros>
                     <output_type>sensor_msgs/LaserScan</output_type>

Commit message: fix sim direction

File: robot_description/urdf/my_robot.xacro (robot description, xacro)
@@ -4,5 +4,5 @@
     <xacro:include filename="$(find robot_description)/my_robot_lidar.xacro" />
     <joint name="lidar_joint" type="fixed">
-        <origin xyz="${-base_radius+lidar_radius} 0 ${base_length+wheel_radius/3}" rpy="0 0 ${PI}" />
+        <origin xyz="${base_radius-lidar_radius} 0 ${base_length+wheel_radius/3}" rpy="0 0 0" />
         <parent link="base_link" />
         <child link="lidar_link" />

File: robot_description/urdf/my_robot_base.xacro (robot description, xacro)
@@ -23,12 +23,13 @@
     <xacro:macro name="wheel" params="prefix reflect">
         <joint name="${prefix}_wheel_joint" type="continuous">
-            <origin xyz="0 ${reflect*wheel_joint_y} ${wheel_radius}" rpy="${PI/2} 0 0" />
+            <!-- <origin xyz="0 ${reflect*wheel_joint_y} ${wheel_radius}" rpy="${PI/2} 0 0" /> -->
+            <origin xyz="0 ${reflect*wheel_joint_y} ${wheel_radius}" rpy="0 0 0" />
             <parent link="base_link"/>
             <child link="${prefix}_wheel_link"/>
-            <axis xyz="0 0 1"/>
+            <axis xyz="0 1 0"/>
         </joint>
         <link name="${prefix}_wheel_link">
             <visual>
-            <origin xyz="0 0 0" rpy="0 0 0" />
+                <origin xyz="0 0 0" rpy="${PI/2} 0 0" />
                 <geometry>
                     <cylinder radius="${wheel_radius}" length = "${wheel_length}"/>
@@ -36,5 +37,5 @@
             </visual>
             <collision>
-            <origin xyz="0 0 0" rpy="0 0 0" />
+                <origin xyz="0 0 0" rpy="${PI/2} 0 0" />
                 <geometry>
                     <cylinder radius="${wheel_radius}" length = "${wheel_length}"/>
