Commit message: add imu sensor

File: src/robot_description/urdf/my_robot.xacro (robot description, xacro)
@@ -3,4 +3,5 @@
     <xacro:include filename="$(find robot_description)/my_robot_base.xacro" />
     <xacro:include filename="$(find robot_description)/my_robot_lidar.xacro" />
+    <xacro:include filename="$(find robot_description)/imu.xacro" />
     <joint name="lidar_joint" type="fixed">
         <origin xyz="${base_radius-lidar_radius} 0 ${base_length+wheel_radius/3}" rpy="0 0 0" />
@@ -8,5 +9,11 @@
         <child link="lidar_link" />
     </joint>
+    <joint name="imu_joint" type="fixed">
+      <parent link="base_link"/>
+      <child link="imu_link"/>
+      <origin xyz="0 0 ${wheel_radius}"/>
+    </joint>
     <xacro:my_robot_base/>
     <xacro:lidar/>
+    <xacro:imu_/>
 </robot>

Commit message: add nav2; modify laser to 360 degree

File: src/robot_description/urdf/my_robot.xacro (robot description, xacro)
@@ -5,5 +5,6 @@
     <xacro:include filename="$(find robot_description)/imu.xacro" />
     <joint name="lidar_joint" type="fixed">
-        <origin xyz="${base_radius-lidar_radius} 0 ${base_length+wheel_radius/3}" rpy="0 0 0" />
+        <!-- <origin xyz="${base_radius-lidar_radius} 0 ${base_length+wheel_radius/3}" rpy="0 0 0" /> -->
+        <origin xyz="0 0 ${base_length+wheel_radius/2}" rpy="0 0 0" />
         <parent link="base_link" />
         <child link="lidar_link" />

File: src/robot_description/urdf/my_robot_base.xacro (robot description, xacro)
@@ -142,5 +142,5 @@
                 <left_joint>left_wheel_joint</left_joint>
                 <right_joint>right_wheel_joint</right_joint>
-                <update_rate>100.0</update_rate>
+                <update_rate>10.0</update_rate>
                 <!-- 表示两个驱动轮的距离, 单位为米 -->
                 <wheel_separation>${wheel_joint_y*2}</wheel_separation>
@@ -161,5 +161,5 @@
                   <argument>--ros-args --remap joint_states:=joint_states</argument>
                 </ros>
-                <update_rate>100</update_rate>
+                <update_rate>10</update_rate>
                 <joint_name>left_wheel_joint</joint_name>
                 <joint_name>right_wheel_joint</joint_name>

File: src/robot_description/urdf/sensors/my_robot_lidar.xacro (robot description, xacro)
@@ -38,6 +38,6 @@
                         <samples>181</samples>
                         <resolution>1</resolution>
-                        <min_angle>-1.046666667</min_angle>
-                        <max_angle>1.04666667</max_angle>
+                        <min_angle>-3.14</min_angle>
+                        <max_angle>3.14</max_angle>
                       </horizontal>
                     </scan>
